File: PCB/Schematics/VNP.sch (EAGLE design)
At the start: 4 parts

Commit message: PCB Push
Parts:
- added 9V-IN: (no value), SparkFun-Connectors:CONN_02PTH3
- added BUZZER: (no value), SparkFun-Connectors:CONN_02LOCK_LONGPADS
- added C5, C6: 10uf, 01_SparkFun:CAP1206
- added U1: VR, eagle_fab:VR_REGULATOR_SOT223
Connections:
- removed net N$6: C2.1, HC-06.2, U$1.VCC, UPDI.1
- new net GND: 9V-IN.2, BUZZER.2, C2.2, C5.1, C6.1, HC-06.2, U$1.GND, U1.GND, UPDI.2
- new net N$3: BUZZER.1, U$1.PA1/SDA/MOSI/AR2
- new net N$8: C2.1, C6.2, HC-06.1, U$1.VCC, U1.OUT, UPDI.1
- net N$1: now also 9V-IN.1, C5.2, U1.IN; no longer C2.2, HC-06.1, U$1.GND, UPDI.2
Changed lines of the file:
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@@
 </variantdefs>
 <classes>
-<class number="0" name="default" width="0" drill="0">
+<class number="0" name="default" width="0.4572" drill="0">
+</class>
+<class number="2" name="vcc" width="0.5588" drill="0">
 </class>
 </classes>
@@
 <part name="HC-06" library="SparkFun-Connectors" deviceset="CONN_04" device="POLAR"/>
 <part name="UPDI" library="SparkFun-Connectors" deviceset="CONN_03" device="SMD_RA_MALE"/>
+<part name="BUZZER" library="SparkFun-Connectors" deviceset="CONN_02" device="LOCK_LONGPADS"/>
+<part name="9V-IN" library="SparkFun-Connectors" deviceset="CONN_02" device="PTH3"/>
+<part name="U1" library="eagle_fab" deviceset="VR_REGULATOR_SOT223" device="" value="VR"/>
+<part name="C5" library="01_SparkFun" deviceset="CAP" device="1206" value="10uf"/>
+<part name="C6" library="01_SparkFun" deviceset="CAP" device="1206" value="10uf"/>
 </parts>
 <sheets>
@@
 <instance part="UPDI" gate="J$1" x="63.5" y="40.64" smashed="yes" rot="R270">
 <attribute name="VALUE" x="56.134" y="43.18" size="1.778" layer="96" font="vector" rot="R270"/>
-<attribute name="NAME" x="69.088" y="43.18" size="1.778" layer="95" font="vector" rot="R270"/>
+<attribute name="NAME" x="63.5" y="43.688" size="1.778" layer="95" font="vector"/>
+</instance>
+<instance part="BUZZER" gate="G$1" x="7.62" y="7.62" smashed="yes" rot="R90">
+<attribute name="VALUE" x="12.446" y="5.08" size="1.778" layer="96" font="vector" rot="R90"/>
+<attribute name="NAME" x="12.7" y="4.572" size="1.778" layer="95" font="vector" rot="R180"/>
+</instance>
+<instance part="9V-IN" gate="G$1" x="-12.7" y="0" smashed="yes">
+<attribute name="VALUE" x="-15.24" y="-4.826" size="1.778" layer="96" font="vector"/>
+<attribute name="NAME" x="-15.24" y="5.588" size="1.778" layer="95" font="vector"/>
+</instance>
+<instance part="U1" gate="G$1" x="17.78" y="-5.08" smashed="yes">
+<attribute name="NAME" x="11.43" y="-11.43" size="1.27" layer="95"/>
+<attribute name="VALUE" x="19.05" y="-11.43" size="1.27" layer="96"/>
+</instance>
+<instance part="C5" gate="G$1" x="0" y="-5.08" smashed="yes" rot="R180">
+<attribute name="NAME" x="-1.524" y="-8.001" size="1.778" layer="95" rot="R180"/>
+<attribute name="VALUE" x="-1.524" y="-2.921" size="1.778" layer="96" rot="R180"/>
+</instance>
+<instance part="C6" gate="G$1" x="38.1" y="-5.08" smashed="yes" rot="R180">
+<attribute name="NAME" x="36.576" y="-8.001" size="1.778" layer="95" rot="R180"/>
+<attribute name="VALUE" x="36.576" y="-2.921" size="1.778" layer="96" rot="R180"/>
 </instance>
 </instances>
@@
 </busses>
 <nets>
-<net name="N$6" class="0">
-<segment>
-<wire x1="0" y1="27.94" x2="7.62" y2="27.94" width="0.1524" layer="91"/>
-<pinref part="HC-06" gate="J1" pin="2"/>
-<wire x1="0" y1="27.94" x2="0" y2="17.78" width="0.1524" layer="91"/>
-<wire x1="0" y1="17.78" x2="-2.54" y2="17.78" width="0.1524" layer="91"/>
-<pinref part="U$1" gate="G$1" pin="VCC"/>
-<wire x1="10.16" y1="22.86" x2="7.62" y2="22.86" width="0.1524" layer="91"/>
-<wire x1="7.62" y1="22.86" x2="7.62" y2="27.94" width="0.1524" layer="91"/>
-<junction x="7.62" y="27.94"/>
-<pinref part="C2" gate="&gt;NAME" pin="1"/>
-<wire x1="7.62" y1="27.94" x2="30.48" y2="27.94" width="0.1524" layer="91"/>
-<wire x1="7.62" y1="27.94" x2="7.62" y2="30.48" width="0.1524" layer="91"/>
-<wire x1="7.62" y1="30.48" x2="60.96" y2="30.48" width="0.1524" layer="91"/>
-<junction x="7.62" y="27.94"/>
-<pinref part="UPDI" gate="J$1" pin="1"/>
-<wire x1="60.96" y1="30.48" x2="60.96" y2="33.02" width="0.1524" layer="91"/>
-</segment>
-</net>
 <net name="N$4" class="0">
 <segment>
@@
 </segment>
 </net>
-<net name="N$1" class="0">
+<net name="N$2" class="0">
 <segment>
-<pinref part="HC-06" gate="J1" pin="1"/>
-<wire x1="-2.54" y1="15.24" x2="0" y2="15.24" width="0.1524" layer="91"/>
+<pinref part="U$1" gate="G$1" pin="PA0/UPDI/AR5"/>
+<pinref part="UPDI" gate="J$1" pin="3"/>
+<wire x1="55.88" y1="17.78" x2="66.04" y2="17.78" width="0.1524" layer="91"/>
+<wire x1="66.04" y1="17.78" x2="66.04" y2="33.02" width="0.1524" layer="91"/>
+</segment>
+</net>
+<net name="N$3" class="0">
+<segment>
+<pinref part="BUZZER" gate="G$1" pin="1"/>
+<pinref part="U$1" gate="G$1" pin="PA1/SDA/MOSI/AR2"/>
+<wire x1="7.62" y1="15.24" x2="10.16" y2="15.24" width="0.1524" layer="91"/>
+</segment>
+</net>
+<net name="GND" class="0">
+<segment>
+<wire x1="-17.78" y1="7.62" x2="-17.78" y2="-12.7" width="0.1524" layer="91"/>
+<pinref part="9V-IN" gate="G$1" pin="2"/>
+<wire x1="-5.08" y1="2.54" x2="-2.54" y2="2.54" width="0.1524" layer="91"/>
+<wire x1="-2.54" y1="2.54" x2="-2.54" y2="5.08" width="0.1524" layer="91"/>
+<wire x1="-2.54" y1="5.08" x2="-2.54" y2="7.62" width="0.1524" layer="91"/>
+<wire x1="-2.54" y1="7.62" x2="-17.78" y2="7.62" width="0.1524" layer="91"/>
 <wire x1="38.1" y1="27.94" x2="58.42" y2="27.94" width="0.1524" layer="91"/>
 <pinref part="C2" gate="&gt;NAME" pin="2"/>
@@
 <wire x1="58.42" y1="27.94" x2="58.42" y2="22.86" width="0.1524" layer="91"/>
 <junction x="58.42" y="22.86"/>
-<wire x1="0" y1="15.24" x2="0" y2="2.54" width="0.1524" layer="91"/>
+<wire x1="0" y1="15.24" x2="0" y2="5.08" width="0.1524" layer="91"/>
+<wire x1="0" y1="5.08" x2="0" y2="2.54" width="0.1524" layer="91"/>
 <wire x1="58.42" y1="27.94" x2="63.5" y2="27.94" width="0.1524" layer="91"/>
 <junction x="58.42" y="27.94"/>
 <pinref part="UPDI" gate="J$1" pin="2"/>
 <wire x1="63.5" y1="27.94" x2="63.5" y2="33.02" width="0.1524" layer="91"/>
+<pinref part="BUZZER" gate="G$1" pin="2"/>
+<wire x1="5.08" y1="15.24" x2="0" y2="15.24" width="0.1524" layer="91"/>
+<wire x1="-2.54" y1="5.08" x2="0" y2="5.08" width="0.1524" layer="91"/>
+<junction x="-2.54" y="5.08"/>
+<junction x="0" y="5.08"/>
+<pinref part="HC-06" gate="J1" pin="2"/>
+<wire x1="-2.54" y1="17.78" x2="0" y2="17.78" width="0.1524" layer="91"/>
+<wire x1="0" y1="17.78" x2="0" y2="15.24" width="0.1524" layer="91"/>
+<junction x="0" y="15.24"/>
+<pinref part="C6" gate="G$1" pin="1"/>
+<wire x1="38.1" y1="-12.7" x2="38.1" y2="-10.16" width="0.1524" layer="91"/>
+<pinref part="C5" gate="G$1" pin="1"/>
+<wire x1="0" y1="-10.16" x2="0" y2="-12.7" width="0.1524" layer="91"/>
+<wire x1="0" y1="-12.7" x2="17.78" y2="-12.7" width="0.1524" layer="91"/>
+<wire x1="17.78" y1="-12.7" x2="38.1" y2="-12.7" width="0.1524" layer="91"/>
+<pinref part="U1" gate="G$1" pin="GND"/>
+<wire x1="17.78" y1="-10.16" x2="17.78" y2="-12.7" width="0.1524" layer="91"/>
+<junction x="17.78" y="-12.7"/>
+<wire x1="0" y1="-12.7" x2="-17.78" y2="-12.7" width="0.1524" layer="91"/>
+<junction x="0" y="-12.7"/>
 </segment>
 </net>
-<net name="N$2" class="0">
+<net name="N$8" class="0">
 <segment>
-<pinref part="U$1" gate="G$1" pin="PA0/UPDI/AR5"/>
-<pinref part="UPDI" gate="J$1" pin="3"/>
-<wire x1="55.88" y1="17.78" x2="66.04" y2="17.78" width="0.1524" layer="91"/>
-<wire x1="66.04" y1="17.78" x2="66.04" y2="33.02" width="0.1524" layer="91"/>
+<pinref part="C6" gate="G$1" pin="2"/>
+<pinref part="U1" gate="G$1" pin="OUT"/>
+<wire x1="25.4" y1="-2.54" x2="38.1" y2="-2.54" width="0.1524" layer="91"/>
+<junction x="38.1" y="-2.54"/>
+<wire x1="38.1" y1="-2.54" x2="71.12" y2="-2.54" width="0.1524" layer="91"/>
+<wire x1="71.12" y1="-2.54" x2="71.12" y2="45.72" width="0.1524" layer="91"/>
+<pinref part="U$1" gate="G$1" pin="VCC"/>
+<wire x1="10.16" y1="22.86" x2="7.62" y2="22.86" width="0.1524" layer="91"/>
+<wire x1="7.62" y1="22.86" x2="7.62" y2="27.94" width="0.1524" layer="91"/>
+<junction x="7.62" y="27.94"/>
+<pinref part="C2" gate="&gt;NAME" pin="1"/>
+<wire x1="7.62" y1="27.94" x2="30.48" y2="27.94" width="0.1524" layer="91"/>
+<wire x1="7.62" y1="27.94" x2="7.62" y2="30.48" width="0.1524" layer="91"/>
+<wire x1="7.62" y1="30.48" x2="55.88" y2="30.48" width="0.1524" layer="91"/>
+<junction x="7.62" y="27.94"/>
+<pinref part="UPDI" gate="J$1" pin="1"/>
+<wire x1="55.88" y1="30.48" x2="60.96" y2="30.48" width="0.1524" layer="91"/>
+<wire x1="60.96" y1="30.48" x2="60.96" y2="33.02" width="0.1524" layer="91"/>
+<wire x1="71.12" y1="45.72" x2="55.88" y2="45.72" width="0.1524" layer="91"/>
+<wire x1="55.88" y1="45.72" x2="55.88" y2="30.48" width="0.1524" layer="91"/>
+<junction x="55.88" y="30.48"/>
+<pinref part="HC-06" gate="J1" pin="1"/>
+<wire x1="-2.54" y1="15.24" x2="-2.54" y2="10.16" width="0.1524" layer="91"/>
+<wire x1="-2.54" y1="10.16" x2="-17.78" y2="10.16" width="0.1524" layer="91"/>
+<wire x1="-17.78" y1="10.16" x2="-17.78" y2="27.94" width="0.1524" layer="91"/>
+<wire x1="-17.78" y1="27.94" x2="7.62" y2="27.94" width="0.1524" layer="91"/>
 </segment>
 </net>
+<net name="N$1" class="2">
+<segment>
+<pinref part="9V-IN" gate="G$1" pin="1"/>
+<wire x1="-5.08" y1="0" x2="-2.54" y2="0" width="0.1524" layer="91"/>
+<wire x1="-2.54" y1="0" x2="-2.54" y2="-2.54" width="0.1524" layer="91"/>
+<pinref part="U1" gate="G$1" pin="IN"/>
+<pinref part="C5" gate="G$1" pin="2"/>
+<wire x1="0" y1="-2.54" x2="10.16" y2="-2.54" width="0.1524" layer="91"/>
+<wire x1="-2.54" y1="-2.54" x2="0" y2="-2.54" width="0.1524" layer="91"/>
+<junction x="0" y="-2.54"/>
+</segment>
+</net>
