File: CAD/PCB/VNP.brd (EAGLE design)
At the start: 24.8 x 106.7 mm, 10 parts, among them U1 VR

Commit message: PCB Dim Update
Parts:
- moved U$1 6.41 mm to (16.4, 70.4)
- moved U$2 6.41 mm to (9.26, 77.5)
- moved U1 6.41 mm to (10.9, 59.9)
- moved C5 6.41 mm to (21.3, 61.7)
- moved C6 6.41 mm to (24.5, 61.7)
- moved HC-06 6.41 mm to (20.4, 11.3)
- moved 9V-IN 6.41 mm to (25.0, 51.2)
- moved BUZZER 6.41 mm to (15.4, 81.4)
- moved UPDI 6.41 mm to (2.22, 70.3)
- moved C2 6.41 mm to (21.1, 70.3)
Routing:
- net N$21: track 0.00 -> 4.14 mm
- net N$20: track 0.00 -> 2.25 mm
- net N$23: track 0.00 -> 1.50 mm
- net N$22: track 0.00 -> 1.50 mm
Other:
- board size 24.8 x 106.7 mm -> 29.8 x 295.1 mm

Commit message: updates
Routing:
- net N$21: track 4.14 -> 0.00 mm
- net N$20: track 2.25 -> 0.00 mm
- net N$23: track 1.50 -> 0.00 mm
- net N$22: track 1.50 -> 0.00 mm
Other:
- board size 29.8 x 295.1 mm -> 24.8 x 106.7 mm
Changed lines of the file:
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@@
 <wire x1="15.290746875" y1="52.021571875" x2="15.184628125" y2="52.5551125" width="0.001" layer="20"/>
 <hole x="8.078828125" y="7.0555125" drill="3"/>
-<wire x1="0" y1="295.94166875" x2="0" y2="295.677" width="0.001" layer="20"/>
-<wire x1="2.116659375" y1="295.942" x2="1.05833125" y2="294.88366875" width="0.001" layer="20"/>
-<wire x1="1.5875" y1="296.471" x2="0.52916875" y2="295.41266875" width="0.001" layer="20"/>
-<wire x1="1.05833125" y1="297" x2="0" y2="295.94166875" width="0.001" layer="20"/>
-<wire x1="0.79375" y1="297.794" x2="-0.79375" y2="296.206" width="0.001" layer="20"/>
-<wire x1="0" y1="298.323" x2="0" y2="295.942" width="0.001" layer="20"/>
-<wire x1="0" y1="295.942" x2="0" y2="295.94166875" width="0.001" layer="20"/>
-<wire x1="2.116659375" y1="295.942" x2="1.05833125" y2="294.884" width="0.001" layer="20"/>
-<wire x1="1.5875" y1="296.471" x2="0.52916875" y2="295.413" width="0.001" layer="20"/>
-<wire x1="1.05833125" y1="297" x2="0" y2="295.942" width="0.001" layer="20"/>
 <wire x1="9.165821875" y1="95.0740375" x2="8.964871875" y2="95.8240375" width="0.001" layer="20"/>
 <wire x1="8.964871875" y1="95.8240375" x2="8.415840625" y2="96.3730375" width="0.001" layer="20"/>
@@
 <wire x1="25.261990625" y1="74.835709375" x2="26.137" y2="74.835709375" width="0.001" layer="1"/>
 </signal>
-<signal name="N$20">
-<wire x1="0.79375" y1="297.794" x2="-0.79375" y2="296.206" width="0.001" layer="1"/>
-</signal>
-<signal name="N$21">
-<wire x1="0" y1="298.323" x2="0" y2="295.94166875" width="0.001" layer="1"/>
-<wire x1="0" y1="295.94166875" x2="0" y2="295.677" width="0.001" layer="1"/>
-<wire x1="1.05833125" y1="297" x2="0" y2="295.94166875" width="0.001" layer="1"/>
-</signal>
-<signal name="N$22">
-<wire x1="2.116659375" y1="295.942" x2="1.05833125" y2="294.88366875" width="0.001" layer="1"/>
-</signal>
-<signal name="N$23">
-<wire x1="1.5875" y1="296.471" x2="0.52916875" y2="295.41266875" width="0.001" layer="1"/>
-</signal>
 </signals>

Commit message: Board Fix
Parts:
- moved C6 5.13 mm to (20.4, 58.6)
- moved HC-06 5.13 mm to (16.3, 8.14)
- moved BUZZER 5.13 mm to (11.3, 78.2)
- moved C2 5.13 mm to (17.1, 67.2)
- moved UPDI 5.13 mm to (-1.85, 67.2)
- moved 9V-IN 5.13 mm to (20.9, 48.1)
- moved C5 5.13 mm to (17.2, 58.6)
- moved U1 5.13 mm to (6.83, 56.8)
- moved U$1 5.13 mm to (12.3, 67.2)
- moved U$2 5.13 mm to (5.18, 74.4)
Other:
- outline, holes or cut-outs redrawn

Commit message: Final PCB, Gerber Files & Final Reciever Code
Parts:
- added U$3: (no value), SparkFun-Aesthetics:OSHW-LOGO-M
- U$2: device SparkFun-Aesthetics:OSHW-LOGO-L_COPPER -> SparkFun-Aesthetics:OSHW-LOGO-M_COPPER
- moved U$2 99.7 mm to (100.8, 46.1)
- moved 9V-IN 80.6 mm to (101.5, 50.3)
- moved BUZZER 80.6 mm to (91.9, 80.5)
- moved C2 80.6 mm to (97.7, 69.4)
- moved C5 80.6 mm to (97.8, 60.9)
- moved C6 80.6 mm to (101.0, 60.9)
- moved HC-06 80.6 mm to (96.9, 10.4)
- moved U$1 80.6 mm to (92.9, 69.5)
- moved U1 80.6 mm to (87.4, 59.0)
- moved UPDI 80.6 mm to (78.7, 69.5)
Connections:
- net N$1 renamed VCC
- net N$2 renamed UPDI
- net N$3 renamed BUZZER
- net N$8 renamed 5V
- removed net N$4: HC-06.3, U$1.3
- removed net N$5: HC-06.4, U$1.2
- new net RX: HC-06.4, U$1.3
- new net TX: HC-06.3, U$1.2
Routing:
- net RX: track 0.00 -> 100.4 mm
- net N$4: track 110.0 -> 12.6 mm
- net TX: track 0.00 -> 90.0 mm
- net N$5: track 92.5 -> 14.2 mm
- net N$14: track 8.91 -> 30.7 mm
- net N$3: track 0.00 -> 14.2 mm
- net N$8: track 0.00 -> 12.6 mm
- net N$1: track 0.00 -> 8.91 mm
- net N$20: track 0.00 -> 8.25 mm
- net N$2: track 0.00 -> 7.77 mm
- net N$18: track 14.2 -> 8.31 mm
- net N$21: track 0.00 -> 5.35 mm
- net N$16: track 14.2 -> 9.22 mm
- net N$22: track 0.00 -> 2.84 mm
- net N$19: track 12.6 -> 10.4 mm
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Other:
- outline, holes or cut-outs redrawn
- board text added: "-"
- board text added: "10uf"
- board text added: "1uf"
- board text added: "412"
- board text added: "5V"
- board text added: "5V Reg"
- board text added: "GND"
- board text added: "UPDI"
