File: CAD/PCB/VNP.sch (EAGLE design)
At the start: 9 parts, among them U1 VR

Commit message: Final PCB, Gerber Files & Final Reciever Code
Connections:
- net N$1 renamed VCC
- net N$2 renamed UPDI
- net N$3 renamed BUZZER
- net N$8 renamed 5V
- removed net N$4: HC-06.3, U$1.PA7/RXD/AR1
- removed net N$5: HC-06.4, U$1.PA6/TXD/DAC/AR0
- new net RX: HC-06.4, U$1.PA7/RXD/AR1
- new net TX: HC-06.3, U$1.PA6/TXD/DAC/AR0
Changed lines of the file:
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@@
 </busses>
 <nets>
-<net name="N$4" class="0">
+<net name="RX" class="0">
 <segment>
-<pinref part="HC-06" gate="J1" pin="3"/>
-<wire x1="-2.54" y1="20.32" x2="2.54" y2="20.32" width="0.1524" layer="91"/>
-<wire x1="2.54" y1="20.32" x2="2.54" y2="17.78" width="0.1524" layer="91"/>
 <pinref part="U$1" gate="G$1" pin="PA7/RXD/AR1"/>
 <wire x1="2.54" y1="17.78" x2="10.16" y2="17.78" width="0.1524" layer="91"/>
+<pinref part="HC-06" gate="J1" pin="4"/>
+<wire x1="-2.54" y1="22.86" x2="2.54" y2="22.86" width="0.1524" layer="91"/>
+<wire x1="2.54" y1="22.86" x2="2.54" y2="17.78" width="0.1524" layer="91"/>
 </segment>
 </net>
-<net name="N$5" class="0">
+<net name="TX" class="0">
 <segment>
-<pinref part="HC-06" gate="J1" pin="4"/>
-<wire x1="-2.54" y1="22.86" x2="5.08" y2="22.86" width="0.1524" layer="91"/>
-<wire x1="5.08" y1="22.86" x2="5.08" y2="20.32" width="0.1524" layer="91"/>
 <pinref part="U$1" gate="G$1" pin="PA6/TXD/DAC/AR0"/>
-<wire x1="5.08" y1="20.32" x2="10.16" y2="20.32" width="0.1524" layer="91"/>
+<pinref part="HC-06" gate="J1" pin="3"/>
+<wire x1="10.16" y1="20.32" x2="-2.54" y2="20.32" width="0.1524" layer="91"/>
 </segment>
 </net>
-<net name="N$2" class="0">
+<net name="UPDI" class="0">
 <segment>
 <pinref part="U$1" gate="G$1" pin="PA0/UPDI/AR5"/>
@@
 </segment>
 </net>
-<net name="N$3" class="0">
+<net name="BUZZER" class="0">
 <segment>
 <pinref part="BUZZER" gate="G$1" pin="1"/>
@@
 </segment>
 </net>
-<net name="N$8" class="0">
+<net name="5V" class="0">
 <segment>
 <pinref part="C6" gate="G$1" pin="2"/>
@@
 </segment>
 </net>
-<net name="N$1" class="2">
+<net name="VCC" class="2">
 <segment>
 <pinref part="9V-IN" gate="G$1" pin="1"/>
